Commit message: Added sim bringup

File: src/hover_bringup/urdf/hoverpi.urdf.xacro (robot description, xacro)
@@ -1,6 +1,7 @@
 <?xml version="1.0"?>
-<robot name="hoverpi" xmlns:xacro="http://www.ros.org/wiki/xacro">
+<robot name="hoverpi"
+  xmlns:xacro="http://www.ros.org/wiki/xacro">
   <xacro:include filename="$(find hover_bringup)/urdf/wheel.urdf.xacro" />
-<!-- Defining the colors used in this robot -->
+  <!-- Defining the colors used in this robot -->
   <material name="Black">
     <color rgba="0.0 0.0 0.0 1.0"/>
@@ -22,29 +23,32 @@
   <!-- Main body radius and height -->
   <!-- Main Body Cylinder base   -->
-  <property name="base_height" value="0.02" />
-  <property name="base_radius" value="0.15" />
-  <property name="base_mass" value="5" /> <!-- in kg-->
+  <property name="base_height" value="0.04" />
+  <property name="base_radius" value="0.25" />
+  <property name="base_mass" value="20" />
+  <!-- in kg-->
+  <property name="laser_height" value="0.05" />
   <!-- caster wheel radius and height -->
   <!-- caster wheel mass -->
   <property name="caster_f_height" value="0.04" />
-  <property name="caster_f_radius" value="0.025" />
-  <property name="caster_f_mass" value="0.5" /> <!-- in kg-->
+  <property name="caster_f_radius" value="0.040" />
+  <property name="caster_f_mass" value="0.5" />
+  <!-- in kg-->
   <!-- caster wheel radius and height -->
   <!-- caster wheel mass -->
   <property name="caster_b_height" value="0.04" />
-  <property name="caster_b_radius" value="0.025" />
-  <property name="caster_b_mass" value="0.5" /> <!-- in kg-->
+  <property name="caster_b_radius" value="0.040" />
+  <property name="caster_b_mass" value="0.5" />
+  <!-- in kg-->
   <!-- Wheels -->
-  <property name="wheel_mass" value="2.5" /> --> <!-- in kg-->
+  <property name="wheel_mass" value="2.5" />
+  <!-- in kg-->
   <property name="base_x_origin_to_wheel_origin" value="0.25" />
-  <property name="base_y_origin_to_wheel_origin" value="0.3" />
+  <property name="base_y_origin_to_wheel_origin" value="0.55" />
   <property name="base_z_origin_to_wheel_origin" value="0.0" />
   <!-- Hokuyo Laser scanner -->
-  <property name="hokuyo_size" value="0.05" />
+  <property name="laser_size" value="0.05" />
   <!-- Macro for calculating inertia of cylinder -->
   <macro name="cylinder_inertia" params="m r h">
-    <inertia  ixx="${m*(3*r*r+h*h)/12}" ixy = "0" ixz = "0"
-              iyy="${m*(3*r*r+h*h)/12}" iyz = "0"
-              izz="${m*r*r/2}" />
+    <inertia ixx="${m*(3*r*r+h*h)/12}" ixy = "0" ixz = "0" iyy="${m*(3*r*r+h*h)/12}" iyz = "0" izz="${m*r*r/2}" />
   </macro>
   <!-- BASE-FOOTPRINT -->
@@ -54,13 +58,11 @@
       <mass value="0.0001" />
       <origin xyz="0 0 0" />
-      <inertia ixx="0.0001" ixy="0.0" ixz="0.0"
-          iyy="0.0001" iyz="0.0"
-          izz="0.0001" />
-    </inertial>
-    <visual>
-        <origin xyz="0 0 0" rpy="0 0 0" />
-        <geometry>
-            <box size="0.001 0.001 0.001" />
-        </geometry>
+      <inertia ixx="0.0001" ixy="0.0" ixz="0.0" iyy="0.0001" iyz="0.0" izz="0.0001" />
+    </inertial>
+    <visual>
+      <origin xyz="0 0 0" rpy="0 0 0" />
+      <geometry>
+        <box size="0.001 0.001 0.001" />
+      </geometry>
     </visual>
   </link>
@@ -80,10 +82,10 @@
       <origin xyz="0 0 0" />
       <!--The 3x3 rotational inertia matrix. -->
-        <cylinder_inertia  m="${base_mass}" r="${base_radius}" h="${base_height}" />
+      <cylinder_inertia m="${base_mass}" r="${base_radius}" h="${base_height}" />
     </inertial>
     <visual>
       <origin xyz="0 0 0" rpy="0 0 0" />
       <geometry>
-          <cylinder length="${base_height}" radius="${base_radius}" />
+        <cylinder length="${base_height}" radius="${base_radius}" />
       </geometry>
       <material name="White" />
@@ -92,5 +94,5 @@
       <origin xyz="0 0 0" rpy="0 0 0 " />
       <geometry>
-          <cylinder length="${base_height}" radius="${base_radius}" />
+        <cylinder length="${base_height}" radius="${base_radius}" />
       </geometry>
     </collision>
@@ -100,110 +102,106 @@
     <turnGravityOff>false</turnGravityOff>
   </gazebo>
-<!--Caster front  -->
-    <link name="caster_front_link">
+  <!--Caster front  -->
+  <link name="caster_front_link">
     <visual>
       <origin xyz="0 0.02 0" rpy="${M_PI/2} 0 0" />
       <geometry>
-	<sphere radius="${caster_f_radius}" />
+        <sphere radius="${caster_f_radius}" />
       </geometry>
       <material name="Black" />
     </visual>
-      <collision>
-        <geometry>
-	<sphere radius="${caster_f_radius}" />
-        </geometry>
+    <collision>
+      <geometry>
+        <sphere radius="${caster_f_radius}" />
+      </geometry>
       <origin xyz="0 0.02 0" rpy="${M_PI/2} 0 0" />
-      </collision>
-      <inertial>
-        <mass value="${caster_f_mass}" />
-        <origin xyz="0 0 0" />
-        <inertia ixx="0.001" ixy="0.0" ixz="0.0"
-                 iyy="0.001" iyz="0.0"
-                 izz="0.001" />
-      </inertial>
-    </link>
- <joint name="caster_front_joint" type="fixed">
-      <parent link="base_link"/>
-      <child link="caster_front_link"/>
-      <origin xyz="0.115 0.0 0.007" rpy="${-M_PI/2} 0 0"/>
-    </joint>
+    </collision>
+    <inertial>
+      <mass value="${caster_f_mass}" />
+      <origin xyz="0 0 0" />
+      <inertia ixx="0.001" ixy="0.0" ixz="0.0" iyy="0.001" iyz="0.0" izz="0.001" />
+    </inertial>
+  </link>
+  <joint name="caster_front_joint" type="fixed">
+    <parent link="base_link"/>
+    <child link="caster_front_link"/>
+    <origin xyz="0.2 0.0 -0.025" rpy="${-M_PI/2} 0 0"/>
+  </joint>
   <gazebo reference="caster_front_link">
     <turnGravityOff>false</turnGravityOff>
   </gazebo>
-<!--Caster back  -->
-    <link name="caster_back_link">
+  <!--Caster back  -->
+  <link name="caster_back_link">
     <visual>
       <origin xyz="0.02 0.02 0 " rpy="${M_PI/2} 0 0" />
       <geometry>
-	<sphere radius="${caster_b_radius}" />
+        <sphere radius="${caster_b_radius}" />
       </geometry>
       <material name="Black" />
     </visual>
-      <collision>
-        <geometry>
-		<sphere radius="${caster_b_radius}" />
-        </geometry>
+    <collision>
+      <geometry>
+        <sphere radius="${caster_b_radius}" />
+      </geometry>
       <origin xyz="0 0.02 0 " rpy="${M_PI/2} 0 0" />
-      </collision>
-      <inertial>
-        <mass value="${caster_b_mass}" />
-        <origin xyz="0 0 0" />
-        <inertia ixx="0.001" ixy="0.0" ixz="0.0"
-                 iyy="0.001" iyz="0.0"
-                 izz="0.001" />
-      </inertial>
-    </link>
-    <joint name="caster_back_joint" type="fixed">
-      <parent link="base_link"/>
-      <child link="caster_back_link"/>
-      <origin xyz="-0.135 0.0 0.009" rpy="${-M_PI/2} 0 0"/>
-    </joint>
+    </collision>
+    <inertial>
+      <mass value="${caster_b_mass}" />
+      <origin xyz="0 0 0" />
+      <inertia ixx="0.001" ixy="0.0" ixz="0.0" iyy="0.001" iyz="0.0" izz="0.001" />
+    </inertial>
+  </link>
+  <joint name="caster_back_joint" type="fixed">
+    <parent link="base_link"/>
+    <child link="caster_back_link"/>
+    <origin xyz="-0.2 0.0 -0.0250" rpy="${-M_PI/2} 0 0"/>
+  </joint>
   <gazebo reference="caster_back_link">
     <turnGravityOff>false</turnGravityOff>
   </gazebo>
-<!-- Wheel Definitions -->
-  <wheel fb="front" lr="right" parent="base_link" translateX="0" translateY="0.5" flipY="1"/>
-  <wheel fb="front" lr="left" parent="base_link" translateX="0" translateY="-0.5" flipY="1"/>
+  <!-- Wheel Definitions -->
+  <wheel fb="front" lr="right" parent="base_link" translateX="0" translateY="-0.5" flipY="1"/>
+  <wheel fb="front" lr="left" parent="base_link" translateX="0" translateY="0.5" flipY="1"/>
   <!-- SENSORS -->
-  <!-- hokuyo -->
-  <link name="hokuyo_link">
+  <!-- rplidar -->
+  <link name="base_laser_link">
     <visual>
       <origin xyz="0 0 0" rpy="0 0 0" />
       <geometry>
-        <box size="${hokuyo_size} ${hokuyo_size} ${hokuyo_size}"/>
+        <box size="${laser_size} ${laser_size} ${laser_size}"/>
       </geometry>
       <material name="Blue" />
     </visual>
   </link>
-  <joint name="hokuyo_joint" type="fixed">
-    <origin xyz="${base_radius - hokuyo_size/2} 0 ${base_height+hokuyo_size/4}" rpy="0 0 0" />
+  <joint name="rplidar_joint" type="fixed">
+    <origin xyz="${ - laser_size/2} 0 ${base_height+laser_size/4 + laser_height}" rpy="0 0 0" />
     <parent link="base_link"/>
-    <child link="hokuyo_link" />
-  </joint>
-  <gazebo reference="hokuyo_link">
+    <child link="base_laser_link" />
+  </joint>
+  <gazebo reference="base_laser_link">
     <material>Gazebo/Blue</material>
     <turnGravityOff>false</turnGravityOff>
     <sensor type="ray" name="head_hokuyo_sensor">
-      <pose>${hokuyo_size/2} 0 0 0 0 0</pose>
+      <pose>${laser_size/2} 0 0 0 0 0</pose>
       <visualize>false</visualize>
-      <update_rate>40</update_rate>
+      <update_rate>8</update_rate>
       <ray>
         <scan>
           <horizontal>
-            <samples>720</samples>
+            <samples>8000</samples>
             <resolution>1</resolution>
-            <min_angle>-1.570796</min_angle>
-            <max_angle>1.570796</max_angle>
+            <min_angle>-3.1415926535897931</min_angle>
+            <max_angle>3.1415926535897931</max_angle>
           </horizontal>
         </scan>
         <range>
           <min>0.10</min>
-          <max>10.0</max>
+          <max>12.0</max>
           <resolution>0.001</resolution>
         </range>
       </ray>
-      <plugin name="gazebo_ros_head_hokuyo_controller" filename="libgazebo_ros_laser.so">
-        <topicName>/scan</topicName>
-        <frameName>hokuyo_link</frameName>
+      <plugin name="ros_ray_sensor_controller" filename="libgazebo_ros_laser.so">
+        <topicName>/laserscan</topicName>
+        <frameName>base_laser_link</frameName>
       </plugin>
     </sensor>
@@ -216,5 +214,5 @@
       <robotNamespace>/</robotNamespace>
       <publishTf>1</publishTf>
-      <publishWheelJointState>false</publishWheelJointState>
+      <publishWheelJointState>true</publishWheelJointState>
       <alwaysOn>true</alwaysOn>
       <updateRate>100.0</updateRate>

File: src/hover_bringup/urdf/wheel.urdf.xacro (robot description, xacro)
@@ -1,17 +1,17 @@
 <?xml version="1.0"?>
-<robot name="wheel" xmlns:xacro="http://www.ros.org/wiki/xacro">
+<robot name="wheel"
+  xmlns:xacro="http://www.ros.org/wiki/xacro">
   <!-- Wheels -->
-  <property name="wheel_radius" value="0.04" />
-  <property name="wheel_height" value="0.02" />
-  <property name="wheel_mass" value="2.5" /> <!-- in kg-->
-  <property name="base_x_origin_to_wheel_origin" value="0.25" />
-  <property name="base_y_origin_to_wheel_origin" value="0.3" />
+  <property name="wheel_radius" value="0.09" />
+  <property name="wheel_height" value="0.05" />
+  <property name="wheel_mass" value="2.5" />
+  <!-- in kg-->
+  <property name="base_x_origin_to_wheel_origin" value="0" />
+  <property name="base_y_origin_to_wheel_origin" value="0" />
   <property name="base_z_origin_to_wheel_origin" value="0.0" />
   <macro name="cylinder_inertia" params="m r h">
-    <inertia  ixx="${m*(3*r*r+h*h)/12}" ixy = "0" ixz = "0"
-              iyy="${m*(3*r*r+h*h)/12}" iyz = "0"
-              izz="${m*r*r/2}" />
+    <inertia ixx="${m*(3*r*r+h*h)/12}" ixy = "0" ixz = "0" iyy="${m*(3*r*r+h*h)/12}" iyz = "0" izz="${m*r*r/2}" />
   </macro>
-  <xacro:macro name="wheel" params="fb lr parent translateX translateY flipY"> <!--fb : front, back ; lr: left, right -->
+  <xacro:macro name="wheel" params="fb lr parent translateX translateY flipY">    <!--fb : front, back ; lr: left, right -->
     <link name="${fb}_${lr}_wheel">
       <visual>
@@ -31,5 +31,5 @@
         <mass value="${wheel_mass}" />
         <origin xyz="0 0 0" />
-        <cylinder_inertia  m="${wheel_mass}" r="${wheel_radius}" h="${wheel_height}" />
+        <cylinder_inertia m="${wheel_mass}" r="${wheel_radius}" h="${wheel_height}" />
       </inertial>
     </link>
@@ -37,6 +37,6 @@
       <mu1 value="1.0"/>
       <mu2 value="1.0"/>
-      <kp  value="10000000.0" />
-      <kd  value="1.0" />
+      <kp value="10000000.0" />
+      <kd value="1.0" />
       <fdir1 value="1 0 0"/>
       <material>Gazebo/Grey</material>

Commit message: fixed xacro issues with naming

File: src/hover_bringup/urdf/hoverpi.urdf.xacro (robot description, xacro)
@@ -18,52 +18,41 @@
   <!-- PROPERTY LIST -->
   <!--All units in m-kg-s-radians unit system -->
-  <property name="M_PI" value="3.1415926535897931" />
-  <property name="M_PI_2" value="1.570796327" />
-  <property name="DEG_TO_RAD" value="0.017453293" />
+  <xacro:property name="M_PI" value="3.1415926535897931" />
+  <xacro:property name="M_PI_2" value="1.570796327" />
+  <xacro:property name="DEG_TO_RAD" value="0.017453293" />
   <!-- Main body radius and height -->
   <!-- Main Body Cylinder base   -->
-  <property name="base_height" value="0.04" />
-  <property name="base_radius" value="0.25" />
-  <property name="base_mass" value="20" />
-  <!-- in kg-->
-  <property name="laser_height" value="0.05" />
+  <xacro:property name="base_height" value="0.04" />
+  <xacro:property name="base_radius" value="0.25" />
+  <xacro:property name="base_mass" value="20" />
+  <!-- in kg-->
+  <xacro:property name="laser_height" value="0.05" />
   <!-- caster wheel radius and height -->
   <!-- caster wheel mass -->
-  <property name="caster_f_height" value="0.04" />
-  <property name="caster_f_radius" value="0.040" />
-  <property name="caster_f_mass" value="0.5" />
+  <xacro:property name="caster_f_height" value="0.04" />
+  <xacro:property name="caster_f_radius" value="0.040" />
+  <xacro:property name="caster_f_mass" value="0.5" />
   <!-- in kg-->
   <!-- caster wheel radius and height -->
   <!-- caster wheel mass -->
-  <property name="caster_b_height" value="0.04" />
-  <property name="caster_b_radius" value="0.040" />
-  <property name="caster_b_mass" value="0.5" />
+  <xacro:property name="caster_b_height" value="0.04" />
+  <xacro:property name="caster_b_radius" value="0.040" />
+  <xacro:property name="caster_b_mass" value="0.5" />
   <!-- in kg-->
   <!-- Wheels -->
-  <property name="wheel_mass" value="2.5" />
-  <!-- in kg-->
-  <property name="base_x_origin_to_wheel_origin" value="0.25" />
-  <property name="base_y_origin_to_wheel_origin" value="0.55" />
-  <property name="base_z_origin_to_wheel_origin" value="0.0" />
+  <xacro:property name="wheel_mass" value="2.5" />
+  <!-- in kg-->
+  <xacro:property name="base_x_origin_to_wheel_origin" value="0.25" />
+  <xacro:property name="base_y_origin_to_wheel_origin" value="0.55" />
+  <xacro:property name="base_z_origin_to_wheel_origin" value="0.0" />
   <!-- Hokuyo Laser scanner -->
-  <property name="laser_size" value="0.05" />
+  <xacro:property name="laser_size" value="0.05" />
   <!-- Macro for calculating inertia of cylinder -->
-  <macro name="cylinder_inertia" params="m r h">
+  <xacro:macro name="cylinder_inertia" params="m r h">
     <inertia ixx="${m*(3*r*r+h*h)/12}" ixy = "0" ixz = "0" iyy="${m*(3*r*r+h*h)/12}" iyz = "0" izz="${m*r*r/2}" />
-  </macro>
+  </xacro:macro>
   <!-- BASE-FOOTPRINT -->
   <!-- base_footprint is a fictitious link(frame) that is on the ground right below base_link origin -->
   <link name="base_footprint">
-    <inertial>
-      <mass value="0.0001" />
-      <origin xyz="0 0 0" />
-      <inertia ixx="0.0001" ixy="0.0" ixz="0.0" iyy="0.0001" iyz="0.0" izz="0.0001" />
-    </inertial>
-    <visual>
-      <origin xyz="0 0 0" rpy="0 0 0" />
-      <geometry>
-        <box size="0.001 0.001 0.001" />
-      </geometry>
-    </visual>
   </link>
   <gazebo reference="base_footprint">

File: src/hover_bringup/urdf/wheel.urdf.xacro (robot description, xacro)
@@ -3,14 +3,14 @@
   xmlns:xacro="http://www.ros.org/wiki/xacro">
   <!-- Wheels -->
-  <property name="wheel_radius" value="0.09" />
-  <property name="wheel_height" value="0.05" />
-  <property name="wheel_mass" value="2.5" />
+  <xacro:property name="wheel_radius" value="0.09" />
+  <xacro:property name="wheel_height" value="0.05" />
+  <xacro:property name="wheel_mass" value="2.5" />
   <!-- in kg-->
-  <property name="base_x_origin_to_wheel_origin" value="0" />
-  <property name="base_y_origin_to_wheel_origin" value="0" />
-  <property name="base_z_origin_to_wheel_origin" value="0.0" />
-  <macro name="cylinder_inertia" params="m r h">
+  <xacro:property name="base_x_origin_to_wheel_origin" value="0" />
+  <xacro:property name="base_y_origin_to_wheel_origin" value="0" />
+  <xacro:property name="base_z_origin_to_wheel_origin" value="0.0" />
+  <xacro:macro name="cylinder_inertia" params="m r h">
     <inertia ixx="${m*(3*r*r+h*h)/12}" ixy = "0" ixz = "0" iyy="${m*(3*r*r+h*h)/12}" iyz = "0" izz="${m*r*r/2}" />
-  </macro>
+  </xacro:macro>
   <xacro:macro name="wheel" params="fb lr parent translateX translateY flipY">    <!--fb : front, back ; lr: left, right -->
     <link name="${fb}_${lr}_wheel">

Commit message: now publishing wheel joint angle tf

File: src/hover_bringup/urdf/hoverpi.urdf.xacro (robot description, xacro)
@@ -150,6 +150,6 @@
   </gazebo>
   <!-- Wheel Definitions -->
-  <wheel fb="front" lr="right" parent="base_link" translateX="0" translateY="-0.5" flipY="1"/>
-  <wheel fb="front" lr="left" parent="base_link" translateX="0" translateY="0.5" flipY="1"/>
+  <wheel lr="right" parent="base_link" translateX="0" translateY="-0.5" flipY="1"/>
+  <wheel lr="left" parent="base_link" translateX="0" translateY="0.5" flipY="1"/>
   <!-- SENSORS -->
   <!-- rplidar -->

File: src/hover_bringup/urdf/wheel.urdf.xacro (robot description, xacro)
@@ -13,6 +13,6 @@
     <inertia ixx="${m*(3*r*r+h*h)/12}" ixy = "0" ixz = "0" iyy="${m*(3*r*r+h*h)/12}" iyz = "0" izz="${m*r*r/2}" />
   </xacro:macro>
-  <xacro:macro name="wheel" params="fb lr parent translateX translateY flipY">    <!--fb : front, back ; lr: left, right -->
-    <link name="${fb}_${lr}_wheel">
+  <xacro:macro name="wheel" params=" lr parent translateX translateY flipY">    <!--lr: left, right -->
+    <link name="${lr}_wheel">
       <visual>
         <origin xyz="0 0 0" rpy="${flipY*M_PI/2} 0  0 " />
@@ -34,5 +34,5 @@
       </inertial>
     </link>
-    <gazebo reference="${fb}_${lr}_wheel">
+    <gazebo reference="${lr}_wheel">
       <mu1 value="1.0"/>
       <mu2 value="1.0"/>
@@ -43,7 +43,7 @@
       <turnGravityOff>false</turnGravityOff>
     </gazebo>
-    <joint name="${fb}_${lr}_wheel_joint" type="continuous">
+    <joint name="${lr}_wheel_joint" type="continuous">
       <parent link="${parent}"/>
-      <child link="${fb}_${lr}_wheel"/>
+      <child link="${lr}_wheel"/>
       <origin xyz="${translateX * base_x_origin_to_wheel_origin} ${translateY * base_y_origin_to_wheel_origin} ${base_z_origin_to_wheel_origin}" rpy="0 0 0" />
       <axis xyz="0 1 0" rpy="0  0" />
@@ -52,8 +52,8 @@
     </joint>
     <!-- Transmission is important to link the joints and the controller -->
-    <transmission name="${fb}_${lr}_wheel_joint_trans">
+    <transmission name="${lr}_wheel_joint_trans">
       <type>transmission_interface/SimpleTransmission</type>
-      <joint name="${fb}_${lr}_wheel_joint" />
-      <actuator name="${fb}_${lr}_wheel_joint_motor">
+      <joint name="${lr}_wheel_joint" />
+      <actuator name="${lr}_wheel_joint_motor">
         <hardwareInterface>EffortJointInterface</hardwareInterface>
         <mechanicalReduction>1</mechanicalReduction>

Commit message: Adapted laser height

File: src/hover_bringup/urdf/hoverpi.urdf.xacro (robot description, xacro)
@@ -27,5 +27,5 @@
   <xacro:property name="base_mass" value="20" />
   <!-- in kg-->
-  <xacro:property name="laser_height" value="0.05" />
+  <xacro:property name="laser_height" value="0.30" />
   <!-- caster wheel radius and height -->
   <!-- caster wheel mass -->

Commit message: shifted laser by 180 degrees

File: src/hover_bringup/urdf/hoverpi.urdf.xacro (robot description, xacro)
@@ -164,10 +164,10 @@
   </link>
   <joint name="rplidar_joint" type="fixed">
-    <origin xyz="${ - laser_size/2} 0 ${base_height+laser_size/4 + laser_height}" rpy="0 0 0" />
+    <origin xyz="${ - laser_size/2} 0 ${base_height+laser_size/4 + laser_height}" rpy="0 0 ${M_PI}" />
     <parent link="base_link"/>
     <child link="base_laser_link" />
   </joint>
   <gazebo reference="base_laser_link">
-    <material>Gazebo/Blue</material>
+    <material>Gazebo/Blue</material>)
     <turnGravityOff>false</turnGravityOff>
     <sensor type="ray" name="head_hokuyo_sensor">

Commit message: changed laserscan layout

File: src/hover_bringup/urdf/hoverpi.urdf.xacro (robot description, xacro)
@@ -164,5 +164,5 @@
   </link>
   <joint name="rplidar_joint" type="fixed">
-    <origin xyz="${ - laser_size/2} 0 ${base_height+laser_size/4 + laser_height}" rpy="0 0 ${M_PI}" />
+    <origin xyz="${ - laser_size/2} 0 ${base_height+laser_size/4 + laser_height}" rpy="0 0 0" />
     <parent link="base_link"/>
     <child link="base_laser_link" />
